File: pcb/totem_he.kicad_pcb (KiCad board)
At the start: 2 copper layers, 264.8 x 103 mm, 56 parts

Commit message: Tot-HE-m: routed board, Ergogen modules, final firmware, foam mold
Board
- Ergogen footprint modules for the switch/sensor, mux, XIAO, TRRS and holes; build.sh regenerates the board
  from the case geometry and mux_map.json
- Hand routing from routes.py with the route.py tool: signals on the underside, power as two combs on top
- Silkscreen outlines and labels, board text, field-line artwork and the cat (art.py, art/)
- panel.py and gerbers.sh: both halves joined by snap-off tabs, Gerbers and drill files for JLCPCB

Firmware
- Pin and channel maps regenerated from the routed board; USB name Tot-HE-m; UF2s rebuilt

Case
- PCB mock updated to the final part positions
- foam_mold.scad: two-part mold for the silicone foam between the PCB and the plate, with STLs

Co-Authored-By: Claude Opus 5.5 <noreply@anthropic.com>
Parts:
- H1, H101, H102, H103, H104, H2, H3, H4: footprint ceoloide:mounting_hole_plated -> totemhe:mounting_hole_plated
- TRRS1, TRRS101: footprint ceoloide:trrs_pj320a -> totemhe:trrs_pj320a
- moved S111 67.6 mm to (233.3, 76.2), turned to -10 degrees
- moved S11 67.6 mm to (31.4, 76.2), turned to 10 degrees
- moved S5 61.4 mm to (106.4, 22.2), turned to 0 degrees
- moved S105 61.4 mm to (158.3, 22.2), turned to 0 degrees
- moved S112 55.5 mm to (215.7, 59.2), turned to -4 degrees
- moved S12 55.5 mm to (49.0, 59.2), turned to 4 degrees
- moved S4 55.5 mm to (87.4, 19.2), turned to 0 degrees
- moved S104 55.5 mm to (177.4, 19.2), turned to 0 degrees
- moved S103 52.0 mm to (196.4, 9.71), turned to 0 degrees
- moved S3 52.0 mm to (68.3, 9.71), turned to 0 degrees
- moved S2 40.5 mm to (46.5, 21.2), turned to 4 degrees
- moved S102 40.5 mm to (218.2, 21.2), turned to -4 degrees
- moved S106 40.5 mm to (236.5, 57.4), turned to -10 degrees
- moved S6 40.5 mm to (28.3, 57.4), turned to 10 degrees
- moved S113 40.1 mm to (196.4, 47.8)
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Connections:
- IC101 pad 1: R/K_RING_TOP -> R/K_RING_HOME
- IC101 pad 12: R/K_PINKY_BOTTOM -> R/K_PINKY_HOME
- IC101 pad 13: R/K_PINKY_HOME -> R/K_OUTER
- IC101 pad 14: R/K_RING_BOTTOM -> R/K_PINKY_BOTTOM
- IC101 pad 15: R/K_RING_HOME -> R/K_RING_BOTTOM
- IC101 pad 2: (no net) -> R/K_RING_TOP
- IC101 pad 4: R/K_PINKY_TOP -> (no net)
- IC101 pad 5: R/K_OUTER -> R/K_PINKY_TOP
- IC102 pad 1: R/K_MIDDLE_TOP -> R/K_INDEX_TOP
- IC102 pad 12: R/K_INDEX_BOTTOM -> R/K_MIDDLE_BOTTOM
- IC102 pad 13: R/K_INDEX_HOME -> (no net)
- IC102 pad 14: (no net) -> R/K_INDEX_BOTTOM
- IC102 pad 15: R/K_INDEX_TOP -> R/K_INDEX_HOME
- IC102 pad 2: R/K_MIDDLE_HOME -> (no net)
- IC102 pad 4: (no net) -> R/K_MIDDLE_TOP
- IC102 pad 5: R/K_MIDDLE_BOTTOM -> R/K_MIDDLE_HOME
- IC103 pad 1: R/K_INNER_TOP -> R/K_THUMB3
- IC103 pad 12: R/K_THUMB3 -> (no net)
- IC103 pad 14: R/K_INNER_BOTTOM -> R/K_THUMB1
- IC103 pad 15: R/K_INNER_HOME -> R/K_THUMB2
- IC103 pad 2: (no net) -> R/K_INNER_TOP
- IC103 pad 4: R/K_THUMB1 -> R/K_INNER_HOME
- IC103 pad 5: R/K_THUMB2 -> R/K_INNER_BOTTOM
- IC2 pad 1: (no net) -> L/K_MIDDLE_HOME
- IC2 pad 13: L/K_INDEX_TOP -> L/K_INDEX_BOTTOM
- IC2 pad 14: L/K_INDEX_BOTTOM -> L/K_MIDDLE_BOTTOM
- IC2 pad 15: L/K_MIDDLE_BOTTOM -> (no net)
- IC2 pad 2: (no net) -> L/K_MIDDLE_TOP
- IC2 pad 4: L/K_MIDDLE_HOME -> (no net)
- IC2 pad 5: L/K_MIDDLE_TOP -> L/K_INDEX_TOP
- IC3 pad 1: (no net) -> L/K_THUMB3
- IC3 pad 12: L/K_INNER_BOTTOM -> L/K_INNER_TOP
- IC3 pad 13: L/K_THUMB3 -> L/K_INNER_HOME
- IC3 pad 14: L/K_THUMB2 -> (no net)
- IC3 pad 15: L/K_THUMB1 -> L/K_INNER_BOTTOM
- IC3 pad 2: (no net) -> L/K_THUMB2
- IC3 pad 4: L/K_INNER_TOP -> L/K_THUMB1
- IC3 pad 5: L/K_INNER_HOME -> (no net)
- MCU1 pad 10: (no net) -> L/SEL1
- MCU1 pad 11: (no net) -> L/SEL2
- MCU1 pad 2: L/ADC_B -> L/ADC_C
- MCU1 pad 3: L/ADC_C -> L/ADC_B
- MCU1 pad 5: L/SEL0 -> (no net)
- MCU1 pad 6: L/SEL1 -> (no net)
- MCU1 pad 7: L/DATA -> (no net)
- MCU1 pad 8: (no net) -> L/DATA
- MCU1 pad 9: L/SEL2 -> L/SEL0
- MCU101 pad 10: (no net) -> R/SEL1
- MCU101 pad 11: (no net) -> R/SEL2
- MCU101 pad 2: R/ADC_B -> R/ADC_C
- MCU101 pad 3: R/ADC_C -> R/ADC_B
- MCU101 pad 5: R/SEL0 -> (no net)
- MCU101 pad 6: R/SEL1 -> (no net)
- MCU101 pad 7: R/DATA -> (no net)
- MCU101 pad 8: (no net) -> R/DATA
- MCU101 pad 9: R/SEL2 -> R/SEL0
- S1 pad 2: L/K_PINKY_BOTTOM -> L/K_PINKY_TOP
- S10 pad 2: L/K_INDEX_BOTTOM -> L/K_INNER_HOME
- S101 pad 2: R/K_PINKY_BOTTOM -> R/K_PINKY_TOP
- S102 pad 2: R/K_PINKY_HOME -> R/K_RING_TOP
- S103 pad 2: R/K_PINKY_TOP -> R/K_MIDDLE_TOP
- S104 pad 2: R/K_RING_BOTTOM -> R/K_INDEX_TOP
- S105 pad 2: R/K_RING_HOME -> R/K_INNER_TOP
- S106 pad 2: R/K_RING_TOP -> R/K_PINKY_HOME
- S107 pad 2: R/K_MIDDLE_BOTTOM -> R/K_RING_HOME
- S109 pad 2: R/K_MIDDLE_TOP -> R/K_INDEX_HOME
- S11 pad 2: L/K_INDEX_HOME -> L/K_PINKY_BOTTOM
- S110 pad 2: R/K_INDEX_BOTTOM -> R/K_INNER_HOME
- S111 pad 2: R/K_INDEX_HOME -> R/K_PINKY_BOTTOM
- S112 pad 2: R/K_INDEX_TOP -> R/K_RING_BOTTOM
- S113 pad 2: R/K_INNER_BOTTOM -> R/K_MIDDLE_BOTTOM
- S114 pad 2: R/K_INNER_HOME -> R/K_INDEX_BOTTOM
- S115 pad 2: R/K_INNER_TOP -> R/K_INNER_BOTTOM
- S12 pad 2: L/K_INDEX_TOP -> L/K_RING_BOTTOM
- S13 pad 2: L/K_INNER_BOTTOM -> L/K_MIDDLE_BOTTOM
- S14 pad 2: L/K_INNER_HOME -> L/K_INDEX_BOTTOM
- S15 pad 2: L/K_INNER_TOP -> L/K_INNER_BOTTOM
- S2 pad 2: L/K_PINKY_HOME -> L/K_RING_TOP
- S3 pad 2: L/K_PINKY_TOP -> L/K_MIDDLE_TOP
- S4 pad 2: L/K_RING_BOTTOM -> L/K_INDEX_TOP
- S5 pad 2: L/K_RING_HOME -> L/K_INNER_TOP
- S6 pad 2: L/K_RING_TOP -> L/K_PINKY_HOME
- S7 pad 2: L/K_MIDDLE_BOTTOM -> L/K_RING_HOME
- S9 pad 2: L/K_MIDDLE_TOP -> L/K_INDEX_HOME
Routing:
- net R/VCC: track 0.00 -> 766.5 mm, vias 0 -> 3
- net L/GND: track 0.00 -> 753.8 mm, vias 0 -> 6
- net R/GND: track 0.00 -> 747.0 mm, vias 0 -> 6
- net L/VCC: track 0.00 -> 701.0 mm, vias 0 -> 3
- net L/SEL2: track 0.00 -> 236.5 mm, vias 0 -> 4
- net R/SEL2: track 0.00 -> 233.9 mm, vias 0 -> 4
- net L/SEL1: track 0.00 -> 233.2 mm, vias 0 -> 4
- net R/SEL1: track 0.00 -> 229.5 mm, vias 0 -> 4
- net L/SEL0: track 0.00 -> 227.7 mm, vias 0 -> 4
- net R/SEL0: track 0.00 -> 225.0 mm, vias 0 -> 4
- net L/ADC_C: track 0.00 -> 161.6 mm
- net R/ADC_C: track 0.00 -> 158.3 mm
- net R/DATA: track 0.00 -> 110.3 mm, vias 0 -> 2
- net L/DATA: track 0.00 -> 109.0 mm
- net L/ADC_B: track 0.00 -> 95.2 mm
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Other:
- board text added: "LEFT · rev 1 · 2026-10"
- board text added: "RIGHT · rev 1 · 2026-10"
- board text added: "TRRS: tip 3V3 · ring 2 DATA · sleeve GND"
- board text added: "Tot-HE-m"
- board text added: "Tot-HE-m LEFT rev 1"
- board text added: "Tot-HE-m RIGHT rev 1"
- board text added: "USB on one half only · plug TRRS with USB out"
- board text added: "hall effect split"
